Commit message: ur5 urdf dae

File: src/robot_mover/urdf/measurement_tool.xacro (robot description, xacro)
@@ -15,5 +15,5 @@
         <geometry>
           <!-- The path to the visual meshes in the package. -->
-          <mesh filename="package://robot_mover/meshes/visual/end_effector.stl"/>
+          <mesh filename="package://robot_mover/meshes/visual/end_effector.dae"/>
         </geometry>
       </visual>
@@ -21,5 +21,5 @@
         <geometry>
           <!-- The path to the collision meshes in the package. -->
-          <mesh filename="package://robot_mover/meshes/collision/end_effector.stl"/>
+          <mesh filename="package://robot_mover/meshes/collision/end_effector.dae"/>
         </geometry>
       </collision>

File: src/robot_mover/urdf/ur5_with_measurement_tool.urdf (robot description, URDF)
Before this commit: robot ur5_with_measurement_tool, 14 links, 13 joints
Links:
- link measurement_tool: geometry collision mesh filename=package://robot_mover/meshes/collision/end_effector.dae; visual mesh filename=package://robot_mover/meshes/visual/end_effector.dae
