Commit message: shit fucking works

File: src/fmauch_universal_robot/ur_description/urdf/inc/ur_macro.xacro (robot description, xacro)
@@ -316,4 +316,33 @@
       <child link="${prefix}tool0"/>
     </joint>
+    <!-- Create a fixed joint with a parameterized name. -->
+    <joint name="measurement_tool_joint" type="fixed">
+      <!-- The parent link must be read from the robot model it is attached to. -->
+      <parent link="${prefix}tool0"/>
+      <child link="measurement_tool"/>
+      <!-- The tool is directly attached to the flange. -->
+      <origin rpy="0 0 0" xyz="0 0 0.001"/>
+    </joint>
+    <link name="measurement_tool">
+      <visual>
+        <geometry>
+          <!-- The path to the visual meshes in the package. -->
+          <mesh filename="package://robot_mover/meshes/visual/end_effector.dae"/>
+        </geometry>
+      </visual>
+      <collision>
+        <geometry>
+          <!-- The path to the collision meshes in the package. -->
+          <mesh filename="package://robot_mover/meshes/collision/end_effector.dae"/>
+        </geometry>
+      </collision>
+    </link>
+    <!-- TCP frame -->
+    <joint name="tcp_joint" type="fixed">
+      <origin rpy="0 0 0" xyz="0 0 0.116"/>
+      <parent link="measurement_tool"/>
+      <child link="tcp"/>
+    </joint>
+    <link name="tcp"/>
   </xacro:macro>
 </robot>

Commit message: ur robot pose

File: src/fmauch_universal_robot/ur_description/urdf/inc/ur_macro.xacro (robot description, xacro)
@@ -328,5 +328,5 @@
         <geometry>
           <!-- The path to the visual meshes in the package. -->
-          <mesh filename="package://robot_mover/meshes/visual/end_effector.dae"/>
+          <mesh filename="package://robot_mover/meshes/visual/Stor-Sugekop.dae"/>
         </geometry>
       </visual>
@@ -334,5 +334,5 @@
         <geometry>
           <!-- The path to the collision meshes in the package. -->
-          <mesh filename="package://robot_mover/meshes/collision/end_effector.dae"/>
+          <mesh filename="package://robot_mover/meshes/collision/Stor-Sugekop.dae"/>
         </geometry>
       </collision>

Commit message: robot working gripper + working workspace

File: src/fmauch_universal_robot/ur_description/urdf/inc/ur_macro.xacro (robot description, xacro)
@@ -312,5 +312,5 @@
     <joint name="${prefix}flange-tool0" type="fixed">
       <!-- default toolframe: X+ left, Y+ up, Z+ front -->
-      <origin xyz="0 0 0" rpy="${pi/2.0} 0 ${pi/2.0}"/>
+      <origin xyz="0.16 0 0" rpy="${pi/2.0} 0 ${pi/2.0}"/>
       <parent link="${prefix}flange"/>
       <child link="${prefix}tool0"/>
@@ -322,5 +322,5 @@
       <child link="measurement_tool"/>
       <!-- The tool is directly attached to the flange. -->
-      <origin rpy="0 0 0" xyz="0 0 0.001"/>
+      <origin rpy="1.57 0 0" xyz="-0.0315 0.0425 -0.159"/>
     </joint>
     <link name="measurement_tool">
@@ -328,5 +328,5 @@
         <geometry>
           <!-- The path to the visual meshes in the package. -->
-          <mesh filename="package://robot_mover/meshes/visual/Stor-Sugekop.dae"/>
+          <mesh filename="package://robot_mover/meshes/visual/end_effector.dae"/>
         </geometry>
       </visual>
@@ -334,5 +334,5 @@
         <geometry>
           <!-- The path to the collision meshes in the package. -->
-          <mesh filename="package://robot_mover/meshes/collision/Stor-Sugekop.dae"/>
+          <mesh filename="package://robot_mover/meshes/collision/end_effector.dae"/>
         </geometry>
       </collision>

File: src/fmauch_universal_robot/ur_description/urdf/ur5_with_measurement_tool.urdf (robot description, URDF)
Before this commit: robot ur5_with_measurement_tool, 14 links, 13 joints
Joints:
- joint flange-tool0: origin xyz=0 0 0 rpy=1.57079632679 0 1.57079632679 -> xyz=0 0 1 rpy=1.57079632679 0 1.57079632679
- joint measurement_tool_joint: origin xyz=0 0 0 rpy=0 0 0 -> xyz=0 0 -1 rpy=0 0 0

Commit message: workspace frame converter

File: src/fmauch_universal_robot/ur_description/urdf/inc/ur_macro.xacro (robot description, xacro)
@@ -312,5 +312,5 @@
     <joint name="${prefix}flange-tool0" type="fixed">
       <!-- default toolframe: X+ left, Y+ up, Z+ front -->
-      <origin xyz="0.16 0 0" rpy="${pi/2.0} 0 ${pi/2.0}"/>
+      <origin xyz="0.045 0.09 -0.09" rpy="${pi/2.0} ${pi/4.0} ${pi/2.0}"/>
       <parent link="${prefix}flange"/>
       <child link="${prefix}tool0"/>
@@ -322,5 +322,5 @@
       <child link="measurement_tool"/>
       <!-- The tool is directly attached to the flange. -->
-      <origin rpy="1.57 0 0" xyz="-0.0315 0.0425 -0.159"/>
+      <origin rpy="0 0 1.57" xyz="0 -0.03 -0.04"/>
     </joint>
     <link name="measurement_tool">
@@ -328,5 +328,5 @@
         <geometry>
           <!-- The path to the visual meshes in the package. -->
-          <mesh filename="package://robot_mover/meshes/visual/end_effector.dae"/>
+          <mesh filename="package://robot_mover/meshes/visual/end_effector.dae" scale="1.0 1.75 1.0"/>
         </geometry>
       </visual>
@@ -334,5 +334,5 @@
         <geometry>
           <!-- The path to the collision meshes in the package. -->
-          <mesh filename="package://robot_mover/meshes/collision/end_effector.dae"/>
+          <mesh filename="package://robot_mover/meshes/collision/end_effector.dae" scale="1.0 1.5 1.0"/>
         </geometry>
       </collision>

Commit message: ros move it stuff

File: src/fmauch_universal_robot/ur_description/urdf/inc/ur_macro.xacro (robot description, xacro)
@@ -322,4 +322,5 @@
       <child link="measurement_tool"/>
       <!-- The tool is directly attached to the flange. -->
+      <!--6.3 x 8.5 x 16 cm-->
       <origin rpy="0 0 1.57" xyz="0 -0.03 -0.04"/>
     </joint>
@@ -328,5 +329,5 @@
         <geometry>
           <!-- The path to the visual meshes in the package. -->
-          <mesh filename="package://robot_mover/meshes/visual/end_effector.dae" scale="1.0 1.75 1.0"/>
+          <mesh filename="package://robot_mover/meshes/visual/end_effector.dae" scale="1.0 1.5375 1.0"/>
         </geometry>
       </visual>
@@ -334,5 +335,5 @@
         <geometry>
           <!-- The path to the collision meshes in the package. -->
-          <mesh filename="package://robot_mover/meshes/collision/end_effector.dae" scale="1.0 1.5 1.0"/>
+          <mesh filename="package://robot_mover/meshes/collision/end_effector.dae" scale="1.0 1.5375 1.0"/>
         </geometry>
       </collision>

Commit message: new gripper added

File: src/fmauch_universal_robot/ur_description/urdf/inc/ur_macro.xacro (robot description, xacro)
@@ -312,5 +312,5 @@
     <joint name="${prefix}flange-tool0" type="fixed">
       <!-- default toolframe: X+ left, Y+ up, Z+ front -->
-      <origin xyz="0.045 0.09 -0.09" rpy="${pi/2.0} ${pi/4.0} ${pi/2.0}"/>
+      <origin xyz="0.117 0.0 0.0" rpy="${pi/2.0} 0 ${pi/2.0}"/>
       <parent link="${prefix}flange"/>
       <child link="${prefix}tool0"/>
@@ -323,5 +323,5 @@
       <!-- The tool is directly attached to the flange. -->
       <!--6.3 x 8.5 x 16 cm-->
-      <origin rpy="0 0 1.57" xyz="0 -0.03 -0.04"/>
+      <origin rpy="1.57 0 0" xyz="-0.044 0.044 -0.116"/>
     </joint>
     <link name="measurement_tool">
@@ -329,5 +329,5 @@
         <geometry>
           <!-- The path to the visual meshes in the package. -->
-          <mesh filename="package://robot_mover/meshes/visual/end_effector.dae" scale="1.0 1.5375 1.0"/>
+          <mesh filename="package://robot_mover/meshes/visual/GripperAssembly.STL" scale="1.0 1.0 1.0"/>
         </geometry>
       </visual>
@@ -335,5 +335,5 @@
         <geometry>
           <!-- The path to the collision meshes in the package. -->
-          <mesh filename="package://robot_mover/meshes/collision/end_effector.dae" scale="1.0 1.5375 1.0"/>
+          <mesh filename="package://robot_mover/meshes/collision/GripperAssembly.STL" scale="1.0 1.0 1.0"/>
         </geometry>
       </collision>
