Commit message: New calibration data for hand eye

File: src/fmauch_universal_robot/ur_description/urdf/inc/ur_macro with vacuum.xacro (robot description, xacro)
@@ -312,5 +312,5 @@
     <joint name="${prefix}flange-tool0" type="fixed">
       <!-- default toolframe: X+ left, Y+ up, Z+ front -->
-      <origin xyz="0.03 0.0 0.0" rpy="${pi/2.0} 0 ${pi/2.0}"/>
+      <origin xyz="0.117 0.0 0.0" rpy="${pi/2.0} 0 ${pi/2.0}"/>
       <parent link="${prefix}flange"/>
       <child link="${prefix}tool0"/>
@@ -323,5 +323,5 @@
       <!-- The tool is directly attached to the flange. -->
       <!--6.3 x 8.5 x 16 cm-->
-      <origin rpy="1.57 0 0" xyz="-0.044 0.044 -0.03"/>
+      <origin rpy="1.57 0 0" xyz="-0.044 0.044 -0.116"/>
     </joint>
     <link name="measurement_tool">
@@ -329,5 +329,5 @@
         <geometry>
           <!-- The path to the visual meshes in the package. -->
-          <mesh filename="package://robot_mover/meshes/visual/GripperAssemblyNoVacuum.STL" scale="1.0 1.0 1.0"/>
+          <mesh filename="package://robot_mover/meshes/visual/GripperAssembly.STL" scale="1.0 1.0 1.0"/>
         </geometry>
       </visual>
@@ -335,5 +335,5 @@
         <geometry>
           <!-- The path to the collision meshes in the package. -->
-          <mesh filename="package://robot_mover/meshes/collision/GripperAssemblyNoVacuum.STL" scale="1.0 1.0 1.0"/>
+          <mesh filename="package://robot_mover/meshes/collision/GripperAssembly.STL" scale="1.0 1.0 1.0"/>
         </geometry>
       </collision>

File: src/fmauch_universal_robot/ur_description/urdf/inc/ur_macro.xacro (robot description, xacro)
@@ -312,5 +312,5 @@
     <joint name="${prefix}flange-tool0" type="fixed">
       <!-- default toolframe: X+ left, Y+ up, Z+ front -->
-      <origin xyz="0.117 0.0 0.0" rpy="${pi/2.0} 0 ${pi/2.0}"/>
+      <origin xyz="0.03 0.0 0.0" rpy="${pi/2.0} 0 ${pi/2.0}"/>
       <parent link="${prefix}flange"/>
       <child link="${prefix}tool0"/>
@@ -323,5 +323,5 @@
       <!-- The tool is directly attached to the flange. -->
       <!--6.3 x 8.5 x 16 cm-->
-      <origin rpy="1.57 0 0" xyz="-0.044 0.044 -0.116"/>
+      <origin rpy="1.57 0 0" xyz="-0.044 0.044 -0.03"/>
     </joint>
     <link name="measurement_tool">
@@ -329,5 +329,5 @@
         <geometry>
           <!-- The path to the visual meshes in the package. -->
-          <mesh filename="package://robot_mover/meshes/visual/GripperAssembly.STL" scale="1.0 1.0 1.0"/>
+          <mesh filename="package://robot_mover/meshes/visual/GripperAssemblyNoVacuum.STL" scale="1.0 1.0 1.0"/>
         </geometry>
       </visual>
@@ -335,5 +335,5 @@
         <geometry>
           <!-- The path to the collision meshes in the package. -->
-          <mesh filename="package://robot_mover/meshes/collision/GripperAssembly.STL" scale="1.0 1.0 1.0"/>
+          <mesh filename="package://robot_mover/meshes/collision/GripperAssemblyNoVacuum.STL" scale="1.0 1.0 1.0"/>
         </geometry>
       </collision>
